Commit message: Reorganização do repositório

File: urdf/ur5e.urdf.xacro (robot description, xacro)
@@ -78,13 +78,13 @@
       <visual>
         <geometry>
-          <mesh filename="package://ur_ufba_webots/urdf/meshes/ur5e/visual/base.dae" />
-        </geometry>
-        <material name="LightGrey">
-          <color rgba="0.7 0.7 0.7 1.0"/>
-        </material>
-      </visual>
-      <collision>
-        <geometry>
-          <mesh filename="package://ur_ufba_webots/urdf/meshes/ur5e/collision/base.stl" />
+          <mesh filename="package://ur5_webots_lar/urdf/meshes/ur5e/visual/base.dae" />
+        </geometry>
+        <material name="LightGrey">
+          <color rgba="0.7 0.7 0.7 1.0"/>
+        </material>
+      </visual>
+      <collision>
+        <geometry>
+          <mesh filename="package://ur5_webots_lar/urdf/meshes/ur5e/collision/base.stl" />
         </geometry>
       </collision>
@@ -115,13 +115,13 @@
       <visual>
         <geometry>
-          <mesh filename="package://ur_ufba_webots/urdf/meshes/ur5e/visual/shoulder.dae" />
-        </geometry>
-        <material name="LightGrey">
-          <color rgba="0.7 0.7 0.7 1.0"/>
-        </material>
-      </visual>
-      <collision>
-        <geometry>
-          <mesh filename="package://ur_ufba_webots/urdf/meshes/ur5e/collision/shoulder.stl" />
+          <mesh filename="package://ur5_webots_lar/urdf/meshes/ur5e/visual/shoulder.dae" />
+        </geometry>
+        <material name="LightGrey">
+          <color rgba="0.7 0.7 0.7 1.0"/>
+        </material>
+      </visual>
+      <collision>
+        <geometry>
+          <mesh filename="package://ur5_webots_lar/urdf/meshes/ur5e/collision/shoulder.stl" />
         </geometry>
       </collision>
@@ -152,13 +152,13 @@
       <visual>
         <geometry>
-          <mesh filename="package://ur_ufba_webots/urdf/meshes/ur5e/visual/upperarm.dae" />
-        </geometry>
-        <material name="LightGrey">
-          <color rgba="0.7 0.7 0.7 1.0"/>
-        </material>
-      </visual>
-      <collision>
-        <geometry>
-          <mesh filename="package://ur_ufba_webots/urdf/meshes/ur5e/collision/upperarm.stl" />
+          <mesh filename="package://ur5_webots_lar/urdf/meshes/ur5e/visual/upperarm.dae" />
+        </geometry>
+        <material name="LightGrey">
+          <color rgba="0.7 0.7 0.7 1.0"/>
+        </material>
+      </visual>
+      <collision>
+        <geometry>
+          <mesh filename="package://ur5_webots_lar/urdf/meshes/ur5e/collision/upperarm.stl" />
         </geometry>
       </collision>
@@ -189,13 +189,13 @@
       <visual>
         <geometry>
-          <mesh filename="package://ur_ufba_webots/urdf/meshes/ur5e/visual/forearm.dae" />
-        </geometry>
-        <material name="LightGrey">
-          <color rgba="0.7 0.7 0.7 1.0"/>
-        </material>
-      </visual>
-      <collision>
-        <geometry>
-          <mesh filename="package://ur_ufba_webots/urdf/meshes/ur5e/collision/forearm.stl" />
+          <mesh filename="package://ur5_webots_lar/urdf/meshes/ur5e/visual/forearm.dae" />
+        </geometry>
+        <material name="LightGrey">
+          <color rgba="0.7 0.7 0.7 1.0"/>
+        </material>
+      </visual>
+      <collision>
+        <geometry>
+          <mesh filename="package://ur5_webots_lar/urdf/meshes/ur5e/collision/forearm.stl" />
         </geometry>
       </collision>
@@ -226,13 +226,13 @@
       <visual>
         <geometry>
-          <mesh filename="package://ur_ufba_webots/urdf/meshes/ur5e/visual/wrist1.dae" />
-        </geometry>
-        <material name="LightGrey">
-          <color rgba="0.7 0.7 0.7 1.0"/>
-        </material>
-      </visual>
-      <collision>
-        <geometry>
-          <mesh filename="package://ur_ufba_webots/urdf/meshes/ur5e/collision/wrist1.stl" />
+          <mesh filename="package://ur5_webots_lar/urdf/meshes/ur5e/visual/wrist1.dae" />
+        </geometry>
+        <material name="LightGrey">
+          <color rgba="0.7 0.7 0.7 1.0"/>
+        </material>
+      </visual>
+      <collision>
+        <geometry>
+          <mesh filename="package://ur5_webots_lar/urdf/meshes/ur5e/collision/wrist1.stl" />
         </geometry>
       </collision>
@@ -263,13 +263,13 @@
       <visual>
         <geometry>
-          <mesh filename="package://ur_ufba_webots/urdf/meshes/ur5e/visual/wrist2.dae" />
-        </geometry>
-        <material name="LightGrey">
-          <color rgba="0.7 0.7 0.7 1.0"/>
-        </material>
-      </visual>
-      <collision>
-        <geometry>
-          <mesh filename="package://ur_ufba_webots/urdf/meshes/ur5e/collision/wrist2.stl" />
+          <mesh filename="package://ur5_webots_lar/urdf/meshes/ur5e/visual/wrist2.dae" />
+        </geometry>
+        <material name="LightGrey">
+          <color rgba="0.7 0.7 0.7 1.0"/>
+        </material>
+      </visual>
+      <collision>
+        <geometry>
+          <mesh filename="package://ur5_webots_lar/urdf/meshes/ur5e/collision/wrist2.stl" />
         </geometry>
       </collision>
@@ -300,13 +300,13 @@
       <visual>
         <geometry>
-          <mesh filename="package://ur_ufba_webots/urdf/meshes/ur5e/visual/wrist3.dae" />
-        </geometry>
-        <material name="LightGrey">
-          <color rgba="0.7 0.7 0.7 1.0"/>
-        </material>
-      </visual>
-      <collision>
-        <geometry>
-          <mesh filename="package://ur_ufba_webots/urdf/meshes/ur5e/collision/wrist3.stl" />
+          <mesh filename="package://ur5_webots_lar/urdf/meshes/ur5e/visual/wrist3.dae" />
+        </geometry>
+        <material name="LightGrey">
+          <color rgba="0.7 0.7 0.7 1.0"/>
+        </material>
+      </visual>
+      <collision>
+        <geometry>
+          <mesh filename="package://ur5_webots_lar/urdf/meshes/ur5e/collision/wrist3.stl" />
         </geometry>
       </collision>

File: urdf/ur5e_joint_limited_robot.urdf.xacro (robot description, xacro)
@@ -2,6 +2,6 @@
 <robot xmlns:xacro="http://ros.org/wiki/xacro" name="ur5e" >
   <!-- ur5e -->
-  <xacro:include filename="$(find ur_ufba_webots)/urdf/ur5e.urdf.xacro" />
-  <xacro:include filename="$(find ur_ufba_webots)/urdf/_d435.urdf.xacro" />
+  <xacro:include filename="$(find ur5_webots_lar)/urdf/ur5e.urdf.xacro" />
+  <xacro:include filename="$(find ur5_webots_lar)/urdf/_d435.urdf.xacro" />
   <!-- arm -->
   <xacro:ur5e_robot prefix="" joint_limited="true"
@@ -56,5 +56,5 @@
       <origin rpy="0 0 0" xyz="0 0 0"/>
       <geometry>
-        <mesh filename="package://ur_ufba_webots/protos/CAM_Support2.stl" scale="1 1 1"/>
+        <mesh filename="package://ur5_webots_lar/protos/CAM_Support2.stl" scale="1 1 1"/>
       </geometry>
       <material name="Cyan">
